File: POVRotateHW/BLE.sch (KiCad schematic (older format))
At the start: 24 parts, among them P2 CONN_01X05, U2 M24M01, U3 LMC6062, U4 CYBLE-022001-00

Commit message: Started work on the POV Rotate layout.
Parts:
- C10, C9: footprint (none) -> Capacitors_SMD:C_0603_HandSoldering
- D7: footprint (none) -> Capacitors_SMD:C_1206_HandSoldering
- R10, R11, R12, R13, R5, R6, R7, R8, R9: footprint (none) -> Resistors_SMD:R_0603_HandSoldering
- U2, U3: footprint (none) -> SMD_Packages:SOIC-8-N
- U4: footprint (none) -> KicadLibrary:CYBLE-022001
- W4, W5, W6, W7, W8, W9: footprint (none) -> Measurement_Points:Measurement_Point_Round-SMD-Pad_Small
Changed lines of the file:
@@
 F 0 "U4" H 5900 2750 60  0000 C CNN
 F 1 "CYBLE-022001-00" H 6000 4550 60  0000 C CNN
-F 2 "" H 6000 4250 60  0001 C CNN
+F 2 "KicadLibrary:CYBLE-022001" H 6000 4250 60  0001 C CNN
 F 3 "" H 6000 4250 60  0001 C CNN
 F 4 "428-3566-PROMO-ND" H 6000 3750 60  0001 C CNN "DIGIKEY"
@@
 F 0 "U2" H 2450 3250 60  0000 C CNN
 F 1 "M24M01" H 2450 4150 60  0000 C CNN
-F 2 "" H 2450 3700 60  0001 C CNN
+F 2 "SMD_Packages:SOIC-8-N" H 2450 3700 60  0001 C CNN
 F 3 "" H 2450 3700 60  0001 C CNN
 F 4 "497-14359-1-ND" H 2450 3700 60  0001 C CNN "DIGIKEY"
@@
 F 0 "R6" V 1780 3250 50  0000 C CNN
 F 1 "4k" V 1700 3250 50  0000 C CNN
-F 2 "" V 1630 3250 50  0000 C CNN
+F 2 "Resistors_SMD:R_0603_HandSoldering" V 1630 3250 50  0001 C CNN
 F 3 "" H 1700 3250 50  0000 C CNN
 	1    1700 3250
@@
 F 0 "R5" V 1480 3250 50  0000 C CNN
 F 1 "4k" V 1400 3250 50  0000 C CNN
-F 2 "" V 1330 3250 50  0000 C CNN
+F 2 "Resistors_SMD:R_0603_HandSoldering" V 1330 3250 50  0001 C CNN
 F 3 "" H 1400 3250 50  0000 C CNN
 	1    1400 3250
@@
 F 0 "C9" H 3175 3800 50  0000 L CNN
 F 1 "0.1u" H 3175 3600 50  0000 L CNN
-F 2 "" H 3188 3550 50  0000 C CNN
+F 2 "Capacitors_SMD:C_0603_HandSoldering" H 3188 3550 50  0001 C CNN
 F 3 "" H 3150 3700 50  0000 C CNN
 	1    3150 3700
@@
 F 0 "W6" H 6850 3270 50  0000 C CNN
 F 1 "P4.0" H 6850 3200 50  0000 C CNN
-F 2 "" H 7050 3000 50  0000 C CNN
+F 2 "Measurement_Points:Measurement_Point_Round-SMD-Pad_Small" H 7050 3000 50  0001 C CNN
 F 3 "" H 7050 3000 50  0000 C CNN
 	1    6850 3000
@@
 F 0 "W7" H 7100 3270 50  0000 C CNN
 F 1 "P4.1" H 7100 3200 50  0000 C CNN
-F 2 "" H 7300 3000 50  0000 C CNN
+F 2 "Measurement_Points:Measurement_Point_Round-SMD-Pad_Small" H 7300 3000 50  0001 C CNN
 F 3 "" H 7300 3000 50  0000 C CNN
 	1    7100 3000
@@
 F 0 "W8" H 7350 3270 50  0000 C CNN
 F 1 "P5.0" H 7350 3200 50  0000 C CNN
-F 2 "" H 7550 3000 50  0000 C CNN
+F 2 "Measurement_Points:Measurement_Point_Round-SMD-Pad_Small" H 7550 3000 50  0001 C CNN
 F 3 "" H 7550 3000 50  0000 C CNN
 	1    7350 3000
@@
 F 0 "W9" H 7600 3270 50  0000 C CNN
 F 1 "P5.1" H 7600 3200 50  0000 C CNN
-F 2 "" H 7800 3000 50  0000 C CNN
+F 2 "Measurement_Points:Measurement_Point_Round-SMD-Pad_Small" H 7800 3000 50  0001 C CNN
 F 3 "" H 7800 3000 50  0000 C CNN
 	1    7600 3000
@@
 F 0 "R7" V 3980 4900 50  0000 C CNN
 F 1 "100k" V 3900 4900 50  0000 C CNN
-F 2 "" V 3830 4900 50  0000 C CNN
+F 2 "Resistors_SMD:R_0603_HandSoldering" V 3830 4900 50  0001 C CNN
 F 3 "" H 3900 4900 50  0000 C CNN
 	1    3900 4900
@@
 F 0 "R8" V 3980 5450 50  0000 C CNN
 F 1 "700k" V 3900 5450 50  0000 C CNN
-F 2 "" V 3830 5450 50  0000 C CNN
+F 2 "Resistors_SMD:R_0603_HandSoldering" V 3830 5450 50  0001 C CNN
 F 3 "" H 3900 5450 50  0000 C CNN
 	1    3900 5450
@@
 F 0 "W5" H 4400 3920 50  0000 C CNN
 F 1 "TEST_1P" H 4400 3850 50  0000 C CNN
-F 2 "" H 4600 3650 50  0000 C CNN
+F 2 "Measurement_Points:Measurement_Point_Round-SMD-Pad_Small" H 4600 3650 50  0001 C CNN
 F 3 "" H 4600 3650 50  0000 C CNN
 	1    4400 3650
@@
 F 0 "U3" H 4250 2000 50  0000 L CNN
 F 1 "LMC6062" H 4250 1600 50  0000 L CNN
-F 2 "" H 4250 1800 50  0000 C CNN
+F 2 "SMD_Packages:SOIC-8-N" H 4250 1800 50  0001 C CNN
 F 3 "" H 4250 1800 50  0000 C CNN
 F 4 "LMC6032IMX/NOPBCT-ND" H 4250 1800 60  0001 C CNN "DIGIKEY"
@@
 F 0 "U3" H 6150 1850 50  0000 L CNN
 F 1 "LMC6062" H 6150 1450 50  0000 L CNN
-F 2 "" H 6150 1650 50  0000 C CNN
+F 2 "SMD_Packages:SOIC-8-N" H 6150 1650 50  0001 C CNN
 F 3 "" H 6150 1650 50  0000 C CNN
 	2    6150 1650
@@
 F 0 "R9" V 4280 1000 50  0000 C CNN
 F 1 "1M" V 4200 1000 50  0000 C CNN
-F 2 "" V 4130 1000 50  0000 C CNN
+F 2 "Resistors_SMD:R_0603_HandSoldering" V 4130 1000 50  0001 C CNN
 F 3 "" H 4200 1000 50  0000 C CNN
 	1    4200 1000
@@
 F 0 "C10" H 4225 850 50  0000 L CNN
 F 1 "3p" H 4225 650 50  0000 L CNN
-F 2 "" H 4238 600 50  0000 C CNN
+F 2 "Capacitors_SMD:C_0603_HandSoldering" H 4238 600 50  0001 C CNN
 F 3 "" H 4200 750 50  0000 C CNN
 	1    4200 750
@@
 F 0 "D7" H 3500 2250 50  0000 C CNN
 F 1 "PD15-21B/TR8" H 3500 2050 50  0000 C CNN
-F 2 "" H 3500 2150 50  0000 C CNN
+F 2 "Capacitors_SMD:C_1206_HandSoldering" H 3500 2150 50  0001 C CNN
 F 3 "" H 3500 2150 50  0000 C CNN
 F 4 "1080-1365-1-ND" H 3500 2150 60  0001 C CNN "DIGIKEY"
@@
 F 0 "R10" V 5030 1800 50  0000 C CNN
 F 1 "6K" V 4950 1800 50  0000 C CNN
-F 2 "" V 4880 1800 50  0000 C CNN
+F 2 "Resistors_SMD:R_0603_HandSoldering" V 4880 1800 50  0001 C CNN
 F 3 "" H 4950 1800 50  0000 C CNN
 	1    4950 1800
@@
 F 0 "R13" V 5530 2150 50  0000 C CNN
 F 1 "100K" V 5450 2150 50  0000 C CNN
-F 2 "" V 5380 2150 50  0000 C CNN
+F 2 "Resistors_SMD:R_0603_HandSoldering" V 5380 2150 50  0001 C CNN
 F 3 "" H 5450 2150 50  0000 C CNN
 	1    5450 2150
@@
 F 0 "R11" V 5430 900 50  0000 C CNN
 F 1 "100k" V 5350 900 50  0000 C CNN
-F 2 "" V 5280 900 50  0000 C CNN
+F 2 "Resistors_SMD:R_0603_HandSoldering" V 5280 900 50  0001 C CNN
 F 3 "" H 5350 900 50  0000 C CNN
 	1    5350 900
@@
 F 0 "R12" V 5430 1300 50  0000 C CNN
 F 1 "100k" V 5350 1300 50  0000 C CNN
-F 2 "" V 5280 1300 50  0000 C CNN
+F 2 "Resistors_SMD:R_0603_HandSoldering" V 5280 1300 50  0001 C CNN
 F 3 "" H 5350 1300 50  0000 C CNN
 	1    5350 1300
@@
 F 0 "W4" H 4100 4470 50  0000 C CNN
 F 1 "P3.6" H 4100 4400 50  0000 C CNN
-F 2 "" H 4300 4200 50  0000 C CNN
+F 2 "Measurement_Points:Measurement_Point_Round-SMD-Pad_Small" H 4300 4200 50  0001 C CNN
 F 3 "" H 4300 4200 50  0000 C CNN
 	1    4100 4200

Commit message: Minor updates based on the actual PCB.
Parts:
- R8: value 700k -> 1M
Changed lines of the file:
@@
 LIBS:contrib
 LIBS:valves
-LIBS:Nickslib
-LIBS:mylib
+LIBS:General
 LIBS:POVRotateHW-cache
 EELAYER 25 0
@@
 P 3900 5450
 F 0 "R8" V 3980 5450 50  0000 C CNN
-F 1 "700k" V 3900 5450 50  0000 C CNN
+F 1 "1M" V 3900 5450 50  0000 C CNN
 F 2 "Resistors_SMD:R_0603_HandSoldering" V 3830 5450 50  0001 C CNN
 F 3 "" H 3900 5450 50  0000 C CNN

Commit message: Rerouting board for RevB
Parts:
- removed W8: P5.0, Measurement_Points:Measurement_Point_Round-SMD-Pad_Small, symbol TEST_1P
- removed W9: P5.1, Measurement_Points:Measurement_Point_Round-SMD-Pad_Small, symbol TEST_1P
Connections:
- net labels added: LE, OE
Changed lines of the file:
@@
-	1    0    0    -1
-$EndComp
-$Comp
-L TEST_1P W8
-U 1 1 5817A60A
-P 7350 3000
-F 0 "W8" H 7350 3270 50  0000 C CNN
-F 1 "P5.0" H 7350 3200 50  0000 C CNN
-F 2 "Measurement_Points:Measurement_Point_Round-SMD-Pad_Small" H 7550 3000 50  0001 C CNN
-F 3 "" H 7550 3000 50  0000 C CNN
-	1    7350 3000
-	1    0    0    -1
-$EndComp
-$Comp
-L TEST_1P W9
-U 1 1 5817A645
-P 7600 3000
-F 0 "W9" H 7600 3270 50  0000 C CNN
-F 1 "P5.1" H 7600 3200 50  0000 C CNN
-F 2 "Measurement_Points:Measurement_Point_Round-SMD-Pad_Small" H 7800 3000 50  0001 C CNN
-F 3 "" H 7800 3000 50  0000 C CNN
-	1    7600 3000
 	1    0    0    -1
 $EndComp
@@
 	6600 3350 7350 3350
 Wire Wire Line
-	7350 3350 7350 3000
-Wire Wire Line
-	6600 3450 7600 3450
-Wire Wire Line
-	7600 3450 7600 3000
+	6600 3450 7850 3450
 $Comp
 L R R7
@@
 Wire Wire Line
 	4100 4300 4100 4200
+Text GLabel 7850 3300 2    60   Input ~ 0
+LE
+Text GLabel 7850 3450 2    60   Input ~ 0
+OE
+Wire Wire Line
+	7850 3300 7350 3300
+Wire Wire Line
+	7350 3300 7350 3350
 $EndSCHEMATC

Commit message: Switched the LED driver to a 24-bit LED driver from ST.
Parts:
- removed W7: P4.1, Measurement_Points:Measurement_Point_Round-SMD-Pad_Small, symbol TEST_1P
Connections:
- net labels added: DG
- wire segments 94 -> 95
Changed lines of the file:
@@
-	1    0    0    -1
-$EndComp
-$Comp
-L TEST_1P W7
-U 1 1 5817A5B8
-P 7100 3000
-F 0 "W7" H 7100 3270 50  0000 C CNN
-F 1 "P4.1" H 7100 3200 50  0000 C CNN
-F 2 "Measurement_Points:Measurement_Point_Round-SMD-Pad_Small" H 7300 3000 50  0001 C CNN
-F 3 "" H 7300 3000 50  0000 C CNN
-	1    7100 3000
 	1    0    0    -1
 $EndComp
@@
 	6850 3100 6850 3000
 Wire Wire Line
-	6600 3200 7100 3200
-Wire Wire Line
-	7100 3200 7100 3000
+	6600 3200 7400 3200
 Wire Wire Line
 	6600 3350 7350 3350
@@
 Wire Wire Line
 	7350 3300 7350 3350
+Text GLabel 7850 3100 2    60   Input ~ 0
+DG
+Wire Wire Line
+	7400 3200 7400 3100
+Wire Wire Line
+	7400 3100 7850 3100
 $EndSCHEMATC

Commit message: Completed layout and updates to silk screen.
Parts:
- D7: footprint Capacitors_SMD:C_1206_HandSoldering -> KicadFootprint:2-SMD_Z-Bend; DIGIKEY 1080-1365-1-ND -> 475-1346-1-ND
- U2: DIGIKEY 497-14359-1-ND -> 497-6351-1-ND
Changed lines of the file:
@@
 F 2 "SMD_Packages:SOIC-8-N" H 2450 3700 60  0001 C CNN
 F 3 "" H 2450 3700 60  0001 C CNN
-F 4 "497-14359-1-ND" H 2450 3700 60  0001 C CNN "DIGIKEY"
+F 4 "497-6351-1-ND" H 2450 3700 60  0001 C CNN "DIGIKEY"
 	1    2450 3700
 	1    0    0    -1
@@
 F 0 "D7" H 3500 2250 50  0000 C CNN
 F 1 "PD15-21B/TR8" H 3500 2050 50  0000 C CNN
-F 2 "Capacitors_SMD:C_1206_HandSoldering" H 3500 2150 50  0001 C CNN
+F 2 "KicadFootprint:2-SMD_Z-Bend" H 3500 2150 50  0001 C CNN
 F 3 "" H 3500 2150 50  0000 C CNN
-F 4 "1080-1365-1-ND" H 3500 2150 60  0001 C CNN "DIGIKEY"
+F 4 "475-1346-1-ND" H 3500 2150 60  0001 C CNN "DIGIKEY"
 	1    3500 2150
 	0    1    1    0
