File: POVRotateHW/BLE.sch (KiCad schematic (older format))
At the start: 21 parts, among them P2 CONN_01X05, U2 M24M01, U3 LMC6062, U4 CYBLE-022001-00

Commit message: Updated schematic and removed some old datasheets.
Parts:
- R7: value 100k -> 1M
- R8: value 1M -> 100K
Changed lines of the file:
@@
 P 3900 4900
 F 0 "R7" V 3980 4900 50  0000 C CNN
-F 1 "100k" V 3900 4900 50  0000 C CNN
+F 1 "1M" V 3900 4900 50  0000 C CNN
 F 2 "Resistors_SMD:R_0603_HandSoldering" V 3830 4900 50  0001 C CNN
 F 3 "" H 3900 4900 50  0000 C CNN
@@
 P 3900 5450
 F 0 "R8" V 3980 5450 50  0000 C CNN
-F 1 "1M" V 3900 5450 50  0000 C CNN
+F 1 "100K" V 3900 5450 50  0000 C CNN
 F 2 "Resistors_SMD:R_0603_HandSoldering" V 3830 5450 50  0001 C CNN
 F 3 "" H 3900 5450 50  0000 C CNN

Commit message: More updates. I have a sydstem that now displays a one second time as well as a crazy pattern.
Parts:
- D8: symbol LED -> LED-RESCUE-POVRotateHW; Digikey (none) -> 475-2709-1-ND; PartNum (none) -> LG L29K-G2J1-24-Z
- U2: PartNum (none) -> M24M01-RMN6TP
- U3: Digikey (none) -> LMC6032IMX/NOPBDKR-ND; PartNum (none) -> LMC6032IMX/NOPB
- U4: PartNum (none) -> CYBLE-022001-00
Changed lines of the file:
@@
 EESchema Schematic File Version 2
+LIBS:POVRotateHW-rescue
 LIBS:power
 LIBS:device
@@
 $EndComp
 $Comp
-L LED D8
+L LED-RESCUE-POVRotateHW D8
 U 1 1 58127B39
 P 9800 3300
+AR Path="/58127B39" Ref="D8"  Part="1"
+AR Path="/5812723F/58127B39" Ref="D8"  Part="1"
 F 0 "D8" H 9800 3400 50  0000 C CNN
 F 1 "LED" H 9800 3200 50  0000 C CNN
 F 2 "LEDs:LED_0603" H 9800 3300 50  0001 C CNN
 F 3 "" H 9800 3300 50  0000 C CNN
+F 4 "475-2709-1-ND" H 9800 3300 60  0001 C CNN "Digikey"
+F 5 "LG L29K-G2J1-24-Z" H 9800 3300 60  0001 C CNN "PartNum"
 	1    9800 3300
 	1    0    0    -1
@@
 F 3 "" H 6000 4250 60  0001 C CNN
 F 4 "428-3566-PROMO-ND" H 6000 3750 60  0001 C CNN "DIGIKEY"
+F 5 "CYBLE-022001-00" H 6000 3750 60  0001 C CNN "PartNum"
 	1    6000 3750
 	1    0    0    -1
@@
 F 3 "" H 2450 3700 60  0001 C CNN
 F 4 "497-6351-1-ND" H 2450 3700 60  0001 C CNN "DIGIKEY"
+F 5 "M24M01-RMN6TP" H 2450 3700 60  0001 C CNN "PartNum"
 	1    2450 3700
 	1    0    0    -1
@@
 F 2 "SMD_Packages:SOIC-8-N" H 6150 1650 50  0001 C CNN
 F 3 "" H 6150 1650 50  0000 C CNN
+F 4 "LMC6032IMX/NOPBDKR-ND" H 6150 1650 60  0001 C CNN "Digikey"
+F 5 "LMC6032IMX/NOPB" H 6150 1650 60  0001 C CNN "PartNum"
 	2    6150 1650
 	1    0    0    -1
