File: POVRotateHW/LEDs.sch (KiCad schematic (older format))
At the start: 18 parts, among them U5 STP24DP05

Commit message: Worked on routing the LEDs.
Changed lines of the file:
@@
 P 2000 2850
 F 0 "W7" H 2000 3120 50  0000 C CNN
-F 1 "TEST_1P" H 2000 3050 50  0000 C CNN
+F 1 "TEST_1P" H 2000 3050 50  0001 C CNN
 F 2 "Measurement_Points:Measurement_Point_Round-SMD-Pad_Small" H 2200 2850 50  0001 C CNN
 F 3 "" H 2200 2850 50  0000 C CNN

Commit message: Completed layout and updates to silk screen.
Parts:
- D9: DIGIKEY (none) -> CLV1A-FKB-CHMKPEHBB7A363CT-ND
- U5: DIGIKEY (none) -> 497-8283-1-ND
Changed lines of the file:
@@
 F 2 "Housings_QFP:TQFP-48_7x7mm_Pitch0.5mm" H 4150 3700 60  0001 C CNN
 F 3 "" H 4150 3700 60  0001 C CNN
+F 4 "497-8283-1-ND" H 4150 3700 60  0001 C CNN "DIGIKEY"
 	1    4150 3700
 	1    0    0    -1
@@
 F 2 "KicadFootprint:CREE_PLCC4" H 6450 1100 50  0001 C CNN
 F 3 "" H 6450 1100 50  0000 C CNN
+F 4 "CLV1A-FKB-CHMKPEHBB7A363CT-ND" H 6500 1150 60  0001 C CNN "DIGIKEY"
 	1    6500 1150
 	1    0    0    -1

Commit message: More updates. I have a sydstem that now displays a one second time as well as a crazy pattern.
Parts:
- D10, D11, D12, D13, D14, D15, D16: symbol LED_RABG -> LED_RABG-RESCUE-POVRotateHW
- D9: symbol LED_RABG -> LED_RABG-RESCUE-POVRotateHW; PartNum (none) -> CLV1A-FKB-CHMKPEHBB7A363
- U5: PartNum (none) -> STP24DP05BTR
Changed lines of the file:
@@
 EESchema Schematic File Version 2
+LIBS:POVRotateHW-rescue
 LIBS:power
 LIBS:device
@@
 F 3 "" H 4150 3700 60  0001 C CNN
 F 4 "497-8283-1-ND" H 4150 3700 60  0001 C CNN "DIGIKEY"
+F 5 "STP24DP05BTR" H 4150 3700 60  0001 C CNN "PartNum"
 	1    4150 3700
 	1    0    0    -1
@@
 Connection ~ 3000 2650
 $Comp
-L LED_RABG D9
+L LED_RABG-RESCUE-POVRotateHW D9
 U 1 1 58485395
 P 6500 1150
+AR Path="/58485395" Ref="D9"  Part="1"
+AR Path="/58127254/58485395" Ref="D9"  Part="1"
 F 0 "D9" H 6575 1500 50  0000 C CNN
 F 1 "LED_RABG" H 6525 800 50  0000 C CNN
@@
 F 3 "" H 6450 1100 50  0000 C CNN
 F 4 "CLV1A-FKB-CHMKPEHBB7A363CT-ND" H 6500 1150 60  0001 C CNN "DIGIKEY"
+F 5 "CLV1A-FKB-CHMKPEHBB7A363" H 6500 1150 60  0001 C CNN "PartNum"
 	1    6500 1150
 	1    0    0    -1
 $EndComp
 $Comp
-L LED_RABG D10
+L LED_RABG-RESCUE-POVRotateHW D10
 U 1 1 58485653
 P 6500 2000
+AR Path="/58485653" Ref="D10"  Part="1"
+AR Path="/58127254/58485653" Ref="D10"  Part="1"
 F 0 "D10" H 6575 2350 50  0000 C CNN
 F 1 "LED_RABG" H 6525 1650 50  0000 C CNN
@@
 $EndComp
 $Comp
-L LED_RABG D11
+L LED_RABG-RESCUE-POVRotateHW D11
 U 1 1 584856FD
 P 6500 2850
+AR Path="/584856FD" Ref="D11"  Part="1"
+AR Path="/58127254/584856FD" Ref="D11"  Part="1"
 F 0 "D11" H 6575 3200 50  0000 C CNN
 F 1 "LED_RABG" H 6525 2500 50  0000 C CNN
@@
 $EndComp
 $Comp
-L LED_RABG D12
+L LED_RABG-RESCUE-POVRotateHW D12
 U 1 1 58485742
 P 6500 3700
+AR Path="/58485742" Ref="D12"  Part="1"
+AR Path="/58127254/58485742" Ref="D12"  Part="1"
 F 0 "D12" H 6575 4050 50  0000 C CNN
 F 1 "LED_RABG" H 6525 3350 50  0000 C CNN
@@
 $EndComp
 $Comp
-L LED_RABG D13
+L LED_RABG-RESCUE-POVRotateHW D13
 U 1 1 58485796
 P 6500 4500
+AR Path="/58485796" Ref="D13"  Part="1"
+AR Path="/58127254/58485796" Ref="D13"  Part="1"
 F 0 "D13" H 6575 4850 50  0000 C CNN
 F 1 "LED_RABG" H 6525 4150 50  0000 C CNN
@@
 $EndComp
 $Comp
-L LED_RABG D14
+L LED_RABG-RESCUE-POVRotateHW D14
 U 1 1 58485825
 P 6500 5300
+AR Path="/58485825" Ref="D14"  Part="1"
+AR Path="/58127254/58485825" Ref="D14"  Part="1"
 F 0 "D14" H 6575 5650 50  0000 C CNN
 F 1 "LED_RABG" H 6525 4950 50  0000 C CNN
@@
 $EndComp
 $Comp
-L LED_RABG D15
+L LED_RABG-RESCUE-POVRotateHW D15
 U 1 1 58485885
 P 6500 6150
+AR Path="/58485885" Ref="D15"  Part="1"
+AR Path="/58127254/58485885" Ref="D15"  Part="1"
 F 0 "D15" H 6575 6500 50  0000 C CNN
 F 1 "LED_RABG" H 6525 5800 50  0000 C CNN
@@
 $EndComp
 $Comp
-L LED_RABG D16
+L LED_RABG-RESCUE-POVRotateHW D16
 U 1 1 584858F0
 P 6500 7000
+AR Path="/584858F0" Ref="D16"  Part="1"
+AR Path="/58127254/584858F0" Ref="D16"  Part="1"
 F 0 "D16" H 6575 7350 50  0000 C CNN
 F 1 "LED_RABG" H 6525 6650 50  0000 C CNN
