File: POVRotateHW/Power.sch (KiCad schematic (older format))
At the start: 25 parts, among them U1 A5970AD

Commit message: Worked on routing the LEDs.
Parts:
- W13, W14: renamed from W?; footprint (none) -> Measurement_Points:Measurement_Point_Round-SMD-Pad_Small
Changed lines of the file:
@@
 PWR
 $Comp
-L TEST_1P W?
+L TEST_1P W14
 U 1 1 584868C9
 P 2150 6200
-F 0 "W?" H 2150 6470 50  0000 C CNN
+F 0 "W14" H 2150 6470 50  0000 C CNN
 F 1 "TEST_1P" H 2150 6400 50  0000 C CNN
-F 2 "" H 2350 6200 50  0000 C CNN
+F 2 "Measurement_Points:Measurement_Point_Round-SMD-Pad_Small" H 2350 6200 50  0001 C CNN
 F 3 "" H 2350 6200 50  0000 C CNN
 	1    2150 6200
@@
 $EndComp
 $Comp
-L TEST_1P W?
+L TEST_1P W13
 U 1 1 58486C45
 P 1650 6250
-F 0 "W?" H 1650 6520 50  0000 C CNN
+F 0 "W13" H 1650 6520 50  0000 C CNN
 F 1 "TEST_1P" H 1650 6450 50  0000 C CNN
-F 2 "" H 1850 6250 50  0000 C CNN
+F 2 "Measurement_Points:Measurement_Point_Round-SMD-Pad_Small" H 1850 6250 50  0001 C CNN
 F 3 "" H 1850 6250 50  0000 C CNN
 	1    1650 6250

Commit message: More updates. I have a sydstem that now displays a one second time as well as a crazy pattern.
Parts:
- C2, C3: PartNum (none) -> EEE-FT1H220AR
- C7, C8: PartNum (none) -> TPSB226K006R0375
- D1, D2, D3, D4, D6: PartNum (none) -> STPS2L40U
- D5: PartNum (none) -> 824520201
- L1: PartNum (none) -> B82476A1104M
- U1: PartNum (none) -> A5970ADTR
Changed lines of the file:
@@
 EESchema Schematic File Version 2
+LIBS:POVRotateHW-rescue
 LIBS:power
 LIBS:device
@@
 F 3 "" H 4300 3600 50  0000 C CNN
 F 4 "732-9779-1-ND" H 4300 3600 60  0001 C CNN "DIGIKEY"
+F 5 "824520201" H 4300 3600 60  0001 C CNN "PartNum"
 	1    4300 3600
 	0    1    1    0
@@
 F 3 "" H 6600 2750 50  0000 C CNN
 F 4 "497-5574-1-ND" H 6600 2750 60  0001 C CNN "DIGIKEY"
+F 5 "STPS2L40U" H 6600 2750 60  0001 C CNN "PartNum"
 	1    6600 2750
 	0    1    1    0
@@
 F 3 "" H 7100 2600 50  0000 C CNN
 F 4 "495-2686-1-ND" V 7100 2600 60  0001 C CNN "Digikey"
+F 5 "B82476A1104M" V 7100 2600 60  0001 C CNN "PartNum"
 	1    7100 2600
 	0    -1   -1   0
@@
 F 3 "" H 7800 2850 50  0000 C CNN
 F 4 "478-9063-1-ND" H 7800 2850 60  0001 C CNN "DIGIKEY"
+F 5 "TPSB226K006R0375" H 7800 2850 60  0001 C CNN "PartNum"
 	1    7800 2850
 	1    0    0    -1
@@
 F 3 "" H 2150 1300 50  0000 C CNN
 F 4 "497-5574-1-ND" H 2150 1300 60  0001 C CNN "DIGIKEY"
+F 5 "STPS2L40U" H 2150 1300 60  0001 C CNN "PartNum"
 	1    2150 1300
 	-1   0    0    1
@@
 F 3 "" H 3200 1600 50  0000 C CNN
 F 4 "PCE5022CT-ND" H 3200 1600 60  0001 C CNN "DIGIKEY"
+F 5 "EEE-FT1H220AR" H 3200 1600 60  0001 C CNN "PartNum"
 	1    3200 1600
 	1    0    0    -1
@@
 F 3 "" H 8050 2850 50  0000 C CNN
 F 4 "478-9063-1-ND" H 8050 2850 60  0001 C CNN "DIGIKEY"
+F 5 "TPSB226K006R0375" H 8050 2850 60  0001 C CNN "PartNum"
 	1    8050 2850
 	1    0    0    -1
@@
 F 3 "" H 2150 1600 50  0000 C CNN
 F 4 "497-5574-1-ND" H 2150 1600 60  0001 C CNN "DIGIKEY"
+F 5 "STPS2L40U" H 2150 1600 60  0001 C CNN "PartNum"
 	1    2150 1600
 	-1   0    0    1
@@
 F 3 "" H 2150 1900 50  0000 C CNN
 F 4 "497-5574-1-ND" H 2150 1900 60  0001 C CNN "DIGIKEY"
+F 5 "STPS2L40U" H 2150 1900 60  0001 C CNN "PartNum"
 	1    2150 1900
 	1    0    0    -1
@@
 F 3 "" H 2150 2200 50  0000 C CNN
 F 4 "497-5574-1-ND" H 2150 2200 60  0001 C CNN "DIGIKEY"
+F 5 "STPS2L40U" H 2150 2200 60  0001 C CNN "PartNum"
 	1    2150 2200
 	1    0    0    -1
@@
 F 3 "" H 3600 1600 50  0000 C CNN
 F 4 "PCE5022CT-ND" H 3600 1600 60  0001 C CNN "DIGIKEY"
+F 5 "EEE-FT1H220AR" H 3600 1600 60  0001 C CNN "PartNum"
 	1    3600 1600
 	1    0    0    -1
@@
 F 3 "" H 5700 2700 60  0000 C CNN
 F 4 "497-10183-1-ND" H 5700 2700 60  0001 C CNN "DIGIKEY"
+F 5 "A5970ADTR" H 5700 2700 60  0001 C CNN "PartNum"
 	1    5700 2700
 	1    0    0    -1
